File: psps.sch (KiCad schematic (older format))
At the start: 26 parts, among them J1 USB_C_Receptacle, J2 Conn_01x03, U1 TLV62585, U2 TLV61046ADB

Commit message: Released PSPS 1.1 to oshpark
Parts:
- removed U1: TLV62585, alvarop:TLV62585PDRLR, symbol alvarop:TLV62585
- added C3, C4: 18pF, Capacitor_SMD:C_0402_1005Metric, symbol Device:C_Small
- added C5, C6, C7, C8: 22uF, Capacitor_SMD:C_0603_1608Metric, symbol Device:C_Small
- added C9: 5.6nF, Capacitor_SMD:C_0402_1005Metric, symbol Device:C_Small
- added L2: 470 nH, alvarop:IHLP1212AEERR47M11, symbol Device:L_Small
- added R7: 120k, Resistor_SMD:R_0402_1005Metric, symbol Device:R_Small
- added R8: 402k, Resistor_SMD:R_0402_1005Metric, symbol Device:R_Small
- added U1: TPS62480, alvarop:TPS62480, symbol alvarop:TPS62480
- C1: value 10uF -> 22uF; DKPN 399-4925-1-ND‎ -> ‎445-14560-1-ND‎; Description CAP CER 10UF 10V X5R 0805 -> CAP CER 22UF 10V X7S 0805; MPN ‎C0805C106K8PACTU‎ -> ‎C2012X7S1A226M125AC‎
- C10: renamed from C3; Description CAP CER 1UF 10V X5R 0603 -> CAP CER 1UF 10V X5R 0603
- C11: renamed from C4; Description CAP CER 1UF 10V X5R 0603 -> CAP CER 1UF 10V X5R 0603
- C12: renamed from C5; Description CAP CER 1UF 10V X5R 0603 -> CAP CER 1UF 10V X5R 0603
- C13: renamed from C6; Description CAP CER 10UF 50V X7R 1210 -> CAP CER 10UF 50V X7R 1210
- C14: renamed from C7; Description CAP CER 10UF 50V X7R 1210 -> CAP CER 10UF 50V X7R 1210
- C2: DKPN 490-14659-1-ND‎ -> ‎445-14560-1-ND‎; Description CAP CER 22UF 6.3V X7T 0805 -> CAP CER 22UF 10V X7S 0805; MPN ‎GRM21BD70J226ME44L‎ -> ‎C2012X7S1A226M125AC‎
- L1: value 1uH -> 470 nH; footprint ultra_librarian:SPM6530T-1R0M120 -> alvarop:IHLP1212AEERR47M11; DKPN ‎445-3880-1-ND‎ -> 541-1330-1-ND‎; Description FIXED IND 1UH 13A 7.81 MOHM -> ‎IHLP1212AEERR47M11‎; MPN ‎SPM6530T-1R0M120‎ -> FIXED IND 470NH 6.7A 15 MOHM SMD
- L3: renamed from L2; DKPN 445-16714-1-ND‎ -> 445-9504-1-ND; Description FIXED IND 10UH 940MA 288 MOHM -> FIXED IND 10UH 700MA 280 MOHM; MPN ‎VLS3015ET-100M-CA‎ -> MLP2520S100MT0S1
- R11: renamed from R9; Description RES SMD 71.5K OHM 1% 1/16W 0402 -> RES SMD 71.5K OHM 1% 1/16W 0402
- R3: value 1M -> 0; DKPN 541-3965-1-ND‎ -> 1276-3480-1-ND; Description RES SMD 1M OHM 1% 1/16W 0402 -> RES SMD 0 OHM JUMPER 1/16W 0402; MPN ‎CRCW04021M00FKEDC‎ -> RC1005J000CS
- R4: value 0 -> 402k; DKPN 1276-3480-1-ND -> 541-402KLCT-ND‎; Description RES SMD 0 OHM JUMPER 1/16W 0402 -> RES SMD 402K OHM 1% 1/16W 0402; MPN RC1005J000CS -> ‎CRCW0402402KFKED‎
- R5: value 332k -> 0; DKPN 311-332KLRCT-ND -> 1276-3480-1-ND; Description RES SMD 332K OHM 1% 1/16W 0402 -> RES SMD 0 OHM JUMPER 1/16W 0402; MPN RC0402FR-07332KL -> RC1005J000CS
- R6: value 100k -> 402k; DKPN 311-100KLRCT-ND -> 541-402KLCT-ND‎; Description RES SMD 100K OHM 1% 1/16W 0402 -> RES SMD 402K OHM 1% 1/16W 0402; MPN RC0402FR-07100KL -> ‎CRCW0402402KFKED‎
- R9: renamed from R7; Description RES SMD 1.1M OHM 1% 1/16W 0402 -> RES SMD 1.1M OHM 1% 1/16W 0402
- renumbered R8 to R10
Connections:
- net +5V: now also C2.1, R3.1, U1.3 (VIN1), U1.9 (VIN2); no longer R4.2
- net 2V6: now also R4.1, R6.2, C3.1, C4.1, C5.1, C6.1, C7.1, C8.1, L2.2, R8.2, U1.16 (VO); no longer C2.1, R3.1, R5.2
- net GND: now also R5.2, C5.2, C6.2, C7.2, C8.2, C9.2, R7.2, U1.1 (PGND1), U1.11 (PGND2), U1.13 (AGND), U1.15 (RS), U1.6 (VSEL); no longer R6.1
- net at R3.2: now also U1.4 (EN)
- net at L1.1: now also U1.2 (SW1)
- net at R5.1: now also U1.8 (MODE); no longer R6.2
- new net: L2.1, U1.10 (SW2)
- new net: C9.1, U1.12 (SS/TR)
- new net: C3.2, C4.2, R4.2, R7.1, U1.14 (FB)
- new net: R8.1, U1.5 (PG)
- new net: R6.1, U1.7 (TG)
